Commit message: local scanner sphere attached

File: urdf/ur10e_with_local_scanner.urdf (robot description, URDF)
Before this commit: robot ur10e_with_local_scanner, 14 links, 13 joints
Links:
- link local_scanner: mass None -> 0.0001; geometry collision sphere radius=0.17; visual sphere radius=0.17

Commit message: implemented fixed self collision

File: urdf/ur10e_with_local_scanner.urdf (robot description, URDF)
Before this commit: robot ur10e_with_local_scanner, 14 links, 13 joints
Links:
- link local_scanner: mass 0.0001 -> 0.8
Joints:
- joint base_link-base_link_inertia: origin xyz=0 0 0 rpy=0 0 3.14159265359 -> xyz=0 0 1 rpy=0 0 3.14159265359
